Commit message: Clean roboarm project files

File: roboarm/urdf/roboarm.urdf.xacro (robot description, xacro)
@@ -10,4 +10,13 @@
     <color rgba="0.9 0.5 0.1 1.0"/>
   </material>
+  <material name="black">
+    <color rgba="0.02 0.02 0.02 1.0"/>
+  </material>
+  <link name="base_footprint"/>
+  <joint name="base_footprint_joint" type="fixed">
+    <parent link="base_footprint"/>
+    <child link="base_link"/>
+    <origin xyz="0 0 0.025" rpy="0 0 0"/>
+  </joint>
   <!-- BASE -->
   <link name="base_link">
@@ -29,20 +38,21 @@
     <parent link="base_link"/>
     <child  link="link1"/>
-    <origin xyz="0 0 0.05" rpy="0 0 0"/>
+    <origin xyz="0 0 0.025" rpy="0 0 0"/>
     <axis xyz="0 0 1"/>
     <limit lower="-3.14" upper="3.14" effort="10" velocity="1.0"/>
   </joint>
-  <!-- LINK 1: Lower Arm -->
+  <!-- LINK 1: Shoulder post -->
   <link name="link1">
     <visual>
-      <origin xyz="0 0 0.1" rpy="0 0 0"/>
-      <geometry><box size="0.05 0.05 0.2"/></geometry>
+      <origin xyz="0 0 0.125" rpy="0 0 0"/>
+      <geometry><box size="0.055 0.055 0.25"/></geometry>
       <material name="blue"/>
     </visual>
     <collision>
-      <origin xyz="0 0 0.1" rpy="0 0 0"/>
-      <geometry><box size="0.05 0.05 0.2"/></geometry>
+      <origin xyz="0 0 0.125" rpy="0 0 0"/>
+      <geometry><box size="0.055 0.055 0.25"/></geometry>
     </collision>
     <inertial>
+      <origin xyz="0 0 0.125" rpy="0 0 0"/>
       <mass value="0.5"/>
       <inertia ixx="0.005" ixy="0" ixz="0"
@@ -54,5 +64,5 @@
     <parent link="link1"/>
     <child  link="link2"/>
-    <origin xyz="0 0 0.2" rpy="0 0 0"/>
+    <origin xyz="0 0 0.25" rpy="0 0 0"/>
     <axis xyz="0 1 0"/>
     <limit lower="-1.57" upper="1.57" effort="10" velocity="1.0"/>
@@ -61,13 +71,14 @@
   <link name="link2">
     <visual>
-      <origin xyz="0 0 0.1" rpy="0 0 0"/>
-      <geometry><box size="0.04 0.04 0.2"/></geometry>
+      <origin xyz="0.18 0 0" rpy="0 0 0"/>
+      <geometry><box size="0.36 0.045 0.045"/></geometry>
       <material name="blue"/>
     </visual>
     <collision>
-      <origin xyz="0 0 0.1" rpy="0 0 0"/>
-      <geometry><box size="0.04 0.04 0.2"/></geometry>
+      <origin xyz="0.18 0 0" rpy="0 0 0"/>
+      <geometry><box size="0.36 0.045 0.045"/></geometry>
     </collision>
     <inertial>
+      <origin xyz="0.18 0 0" rpy="0 0 0"/>
       <mass value="0.3"/>
       <inertia ixx="0.003" ixy="0" ixz="0"
@@ -79,5 +90,5 @@
     <parent link="link2"/>
     <child  link="link3"/>
-    <origin xyz="0 0 0.2" rpy="0 0 0"/>
+    <origin xyz="0.36 0 0" rpy="0 0 0"/>
     <axis xyz="0 1 0"/>
     <limit lower="-1.57" upper="1.57" effort="10" velocity="1.0"/>
@@ -86,13 +97,19 @@
   <link name="link3">
     <visual>
-      <origin xyz="0 0 0.08" rpy="0 0 0"/>
-      <geometry><box size="0.03 0.03 0.16"/></geometry>
+      <origin xyz="0.14 0 0" rpy="0 0 0"/>
+      <geometry><box size="0.28 0.035 0.035"/></geometry>
       <material name="orange"/>
     </visual>
+    <visual>
+      <origin xyz="0.3 0 0" rpy="0 0 0"/>
+      <geometry><box size="0.045 0.08 0.04"/></geometry>
+      <material name="black"/>
+    </visual>
     <collision>
-      <origin xyz="0 0 0.08" rpy="0 0 0"/>
-      <geometry><box size="0.03 0.03 0.16"/></geometry>
+      <origin xyz="0.14 0 0" rpy="0 0 0"/>
+      <geometry><box size="0.28 0.035 0.035"/></geometry>
     </collision>
     <inertial>
+      <origin xyz="0.14 0 0" rpy="0 0 0"/>
       <mass value="0.2"/>
       <inertia ixx="0.001" ixy="0" ixz="0"
@@ -100,3 +117,33 @@
     </inertial>
   </link>
+  <gazebo>
+    <plugin
+      filename="gz-sim-joint-position-controller-system"
+      name="gz::sim::systems::JointPositionController">
+      <joint_name>base_joint</joint_name>
+      <p_gain>8.0</p_gain>
+      <i_gain>0.0</i_gain>
+      <d_gain>0.5</d_gain>
+    </plugin>
+  </gazebo>
+  <gazebo>
+    <plugin
+      filename="gz-sim-joint-position-controller-system"
+      name="gz::sim::systems::JointPositionController">
+      <joint_name>shoulder_joint</joint_name>
+      <p_gain>12.0</p_gain>
+      <i_gain>0.0</i_gain>
+      <d_gain>0.7</d_gain>
+    </plugin>
+  </gazebo>
+  <gazebo>
+    <plugin
+      filename="gz-sim-joint-position-controller-system"
+      name="gz::sim::systems::JointPositionController">
+      <joint_name>elbow_joint</joint_name>
+      <p_gain>10.0</p_gain>
+      <i_gain>0.0</i_gain>
+      <d_gain>0.5</d_gain>
+    </plugin>
+  </gazebo>
 </robot>
